Commit message: revise the bundled AR tags size and layout after measuring tag's real size in Blender.

File: wamv_gazebo/urdf/ar_tags/ar_tag.xacro (robot description, xacro)
@@ -1,5 +1,5 @@
 <?xml version="1.0"?>
 <robot xmlns:xacro="http://ros.org/wiki/xacro" name="wam-v-ar_tag">
-<xacro:macro name="ar_tag" params="id side:=0.27 position:='0 0 0' orientation:='0 0 0'">
+<xacro:macro name="ar_tag" params="id side:=0.5 position:='0 0 0' orientation:='0 0 0'">
     <!-- Add link -->
     <link name="ar_tag${id}">
@@ -19,5 +19,5 @@
             <geometry>
 <!--                <box size="${side} ${side} 0.02"/>-->
-                <mesh filename="package://wamv_description/models/marker${id}/meshes/Marker${id}.dae"/>
+                <mesh filename="package://wamv_description/models/marker${id}/meshes/Marker${id}.dae" scale="1 1 1"/>
             </geometry>
         </visual>

File: wamv_gazebo/urdf/ar_tags/hori_ar_tags.xacro (robot description, xacro)
@@ -5,9 +5,9 @@
     <xacro:include filename="$(find wamv_gazebo)/urdf/ar_tags/ar_tag.xacro"/>
     <!-- Downward looking, X faces boat front, Y faces boat left, AR tags are equal-sized squares, added from 1st quadrant counter-clockwisely -->
-    <xacro:property name="side" value="0.27" /> <!-- Side length of AR tag -->
+    <xacro:property name="side" value="0.5" /> <!-- Side length of AR tag -->
     <xacro:property name="half_side" value="${side / 2}" /> <!-- Half side length of AR tag -->
     <xacro:property name="height" value="1.3" /> <!-- Height of AR tag w.r.t boat frame -->
-    <xacro:property name="x_margin" value="0.1" /> <!-- Distance between AR tags in x direction -->
-    <xacro:property name="y_margin" value="0.1" /> <!-- Distance between AR tags in y direction -->
+    <xacro:property name="x_margin" value="0" /> <!-- Distance between AR tags in x direction -->
+    <xacro:property name="y_margin" value="0" /> <!-- Distance between AR tags in y direction -->
     <xacro:property name="x_offset" value="-0.4" /> <!-- Overall translation of AR tags w.r.t boat frame in x direction -->
     <xacro:property name="y_offset" value="0" /> <!-- Overall translation of AR tags w.r.t boat frame in y direction -->
